File: TxBoard.kicad_pcb (KiCad board)
At the start: 2 copper layers, 94 x 31.7 mm, 21 parts, among them J1 RCA Socket, Q1 RU1J002YNTCL, SW1 Pull-Up, SW2 Input(Hi-Z)/Output, SW3 High/Low

Commit message: Yet more changes
Compliance and PCB and QRs, oh my!
Parts:
- added G***: LOGO, TixBoard Footprints:qrc, B.Cu at (180.8, 108.6)
- BT1: footprint BC2AAPC:BAT_BC2AAPC -> TixBoard Footprints:BC2AAPC
- J1: footprint KLPX-0848A-2-B:KLPX-0848A-2-B -> TixBoard Footprints:KLPX-0848A
- SW1, SW2, SW3: footprint JS102011SCQN:JS102011SCQN -> TixBoard Footprints:JS102011SCQN
- moved J1 4.50 mm to (188.1, 97.2)
- turned SW1 to -90 degrees
- turned SW2 to -90 degrees
- turned SW3 to -90 degrees
Other:
- board text added: "Copyright QuarterWave Engineering 2023 CERN-OHL-P-2.0 Source: github.com/quarterwave0/TixBoard/"
